Commit message: erro no CPP

File: wave_gazebo/world_models/ocean_waves/model.xacro (robot description, xacro)
@@ -17,7 +17,7 @@
 -->
 <world xmlns:xacro="http://ros.org/wiki/xacro">
-  <xacro:macro name="ocean_waves" params="gain:=100.1 period:=15
+  <xacro:macro name="ocean_waves" params="gain:=0.1 period:=5
                      direction_x:=1.0 direction_y:=0.0
-                     angle:=0.4 scale:=100.5">
+                     angle:=0.4 scale:=1.5">
   <model name='ocean_waves'>
     <static>true</static>
