Commit message: added ocean trash

File: offshore_uav_pack/worlds/offshore_rig.world.xacro (robot description, xacro)
@@ -70,23 +70,76 @@
     </light>
     <!--}-->
+    <!-- Dunes {-->
     <include>
       <uri>model://lake_bottom</uri>
       <pose frame=''>0 0 -18 0 -0 0</pose>
     </include>
+    <!--}-->
+    <!-- Oil rig {-->
     <include>
       <uri>model://oil_rig</uri>
       <pose frame=''>105 80 -8 0 1.5708 3.141593</pose>
     </include>
+    <!--}-->
+    <!-- Pier {-->
     <include>
       <uri>model://pier</uri>
       <pose frame=''>170 180 -14 0 0 0</pose>
     </include>
+    <!--}-->
+    <!-- Square to calibration of cameras {-->
     <include>
       <uri>model://calib_stereo</uri>
       <pose frame=''>140.0 220.0 9.0 0 0 0</pose>
     </include>
-    <!--Waves-->
+    <!--}-->
+    <!-- Beer Bottle {-->
+    <include>
+      <uri>model://beer_bottle</uri>
+      <pose frame=''>0 0 0.0 1.5708 0 0</pose>
+    </include>
+    <!--}-->
+    <!-- Ocean Trash {-->
+    <!-- Cone {-->
+    <include>
+      <uri>model://cone</uri>
+      <pose frame=''>1 0 0.2 0 0 0</pose>
+    </include>
+    <!--}-->
+    <!-- Garbage bag {-->
+    <include>
+      <uri>model://garbage_bag</uri>
+      <pose frame=''>0 1 0.2 0 0 0</pose>
+    </include>
+    <!--}-->
+    <!-- Sphere {-->
+    <include>
+      <uri>model://sphere</uri>
+      <pose frame=''>1 1 0.2 0 0 0</pose>
+    </include>
+    <!--}-->
+    <!-- Square bottle {-->
+    <include>
+      <uri>model://square_bottle</uri>
+      <pose frame=''>2 1 0.2 1.5708 1.5708 0</pose>
+    </include>
+    <!--}-->
+    <!-- Torus {-->
+    <include>
+      <uri>model://torus</uri>
+      <pose frame=''>1 2 0.2 0.0 0 0</pose>
+    </include>
+    <!--}-->
+    <!-- Water bottle {-->
+    <include>
+      <uri>model://water_bottle</uri>
+      <pose frame=''>2 2 0.2 1.5708 0 0</pose>
+    </include>
+    <!--}-->
+    <!--}-->
+    <!--Waves {-->
     <xacro:include filename="$(find offshore_uav_pack)/worlds/ocean_waves/model.xacro"/>
     <xacro:ocean_waves/>
+    <!--}-->
   </world>
 </sdf>

File: wave_gazebo/world_models/ocean_waves/model.xacro (robot description, xacro)
@@ -17,7 +17,7 @@
 -->
 <world xmlns:xacro="http://ros.org/wiki/xacro">
-  <xacro:macro name="ocean_waves" params="gain:=100.1 period:=15
+  <xacro:macro name="ocean_waves" params="gain:=0.1 period:=5
                      direction_x:=1.0 direction_y:=0.0
-                     angle:=0.4 scale:=100.5">
+                     angle:=0.4">
   <model name='ocean_waves'>
     <static>true</static>
@@ -31,6 +31,6 @@
         <period>${period}</period>
         <number>3</number>
-        <scale>${scale}</scale>
-        <gain>${gain}</gain>
+        <scale>1.5</scale>
+	<gain>${gain}</gain>
         <direction>${direction_x} ${direction_y}</direction>
         <angle>${angle}</angle>
@@ -43,14 +43,12 @@
       <visual name="ocean_waves_visual">
         <plugin name="ocean_waves_visual_plugin" filename="libWavefieldVisualPlugin.so">
-          <enableRtt>true</enableRtt>
-          <rttNoise>0.1</rttNoise>
-          <refractOpacity>0.2</refractOpacity>
-          <reflectOpacity>0.2</reflectOpacity>
+          <shallowRefractRatio>0.2</shallowRefractRatio>
+          <envReflectRatio>1.0</envReflectRatio>
           <wave>
             <model>PMS</model>
             <period>${period}</period>
             <number>3</number>
-            <scale>${scale}</scale>
-            <gain>${gain}</gain>
+            <scale>1.5</scale>
+	    <gain>${gain}</gain>
             <direction>${direction_x} ${direction_y}</direction>
             <angle>${angle}</angle>
@@ -62,5 +60,4 @@
         <geometry>
           <mesh>
-            <scale>${scale} ${scale} 1</scale>
             <uri>model://ocean_waves/meshes/mesh.dae</uri>
           </mesh>
@@ -78,5 +75,4 @@
         <geometry>
           <mesh>
-            <scale>${scale} ${scale} 1</scale>
             <uri>model://ocean_waves/meshes/mesh_below.dae</uri>
           </mesh>

File: wave_gazebo/worlds/ocean_buoys.world.xacro (robot description, xacro)
@@ -65,4 +65,10 @@
     </model>
     -->
+    <!-- Add auto generated model with N buoys -->
+    <model name="robotx_2018_qualifying_avoid_obstacles_buoys">
+      <include>
+        <uri>model://robotx_2018_qualifying_avoid_obstacles_buoys</uri>
+      </include>
+    </model>
   </world>
 </sdf>
