Commit message: Big Wave

File: offshore_uav_pack/worlds/ocean_waves/model.xacro (robot description, xacro)
@@ -17,5 +17,5 @@
 -->
 <world xmlns:xacro="http://ros.org/wiki/xacro">
-  <xacro:macro name="ocean_waves" params="gain:=0.1 period:=5
+  <xacro:macro name="ocean_waves" params="gain:=1.0 period:=15
                      direction_x:=1.0 direction_y:=0.0
                      angle:=0.4 scale:=1.5">

File: offshore_uav_pack/worlds/offshore_rig.world.xacro (robot description, xacro)
@@ -71,7 +71,8 @@
     <!--}-->
     <!-- user camera {-->
+    <!-- <pose>140 120 8 0 0.2 5.7</pose> -->
     <gui>
       <camera name="camera">
-        <pose>140 120 8 0 0.2 5.7</pose>
+        <pose>-20 -20 15 0 0.52 0.52</pose>
       </camera>
     </gui>

File: wave_gazebo/world_models/ocean_waves/model.xacro (robot description, xacro)
@@ -17,7 +17,7 @@
 -->
 <world xmlns:xacro="http://ros.org/wiki/xacro">
-  <xacro:macro name="ocean_waves" params="gain:=0.1 period:=5
+  <xacro:macro name="ocean_waves" params="gain:=10.1 period:=15
                      direction_x:=1.0 direction_y:=0.0
-                     angle:=0.4 scale:=1.5">
+                     angle:=0.4 scale:=10.5">
   <model name='ocean_waves'>
     <static>true</static>
